File: clock-pcb/sub-boards/usb-board/usb-board.kicad_pcb (KiCad board)
At the start: 2 copper layers, 13.4 x 20 mm, 5 parts, among them J1 USB4140-GF-0070-C

Commit message: routing
Parts:
- removed R2: 5.1k, Resistor_SMD:R_0402_1005Metric
- removed USB_BOARD1: Conn_01x02_Socket, clock:SHDR2W64P0X250_1X2_740X575X700P
- added D2: ESD5Zxx, Diode_SMD:D_SOD-523, B.Cu at (27.9, 35.6)
- added D3: ESD5Zxx, Diode_SMD:D_SOD-523, B.Cu at (33.0, 35.6)
- added J8: Conn_01x04_Socket, Connector_JST:JST_XH_B4B-XH-AM_1x04_P2.50mm_Vertical, F.Cu at (26.8, 26.9)
- added R3: 5.1k, Resistor_SMD:R_0402_1005Metric, B.Cu at (30.0, 34.8)
- D1, R1: moved to B.Cu
- J1: value USB4140-GF-0070-C -> USB4145-03-0070-C; footprint clock:USB4140GF0070C -> clock:USB4145030070C
- turned D1 to 180 degrees
Routing:
- net DP: track 0.00 -> 17.1 mm, vias 0 -> 2
- net DN: track 0.00 -> 16.0 mm
- net VBUS: track 15.4 -> 23.4 mm, vias 1 -> 0
- net Net-(J1-CC2): track 2.71 -> 5.73 mm, vias 1 -> 2
- net Net-(J1-CC1): track 2.71 -> 5.64 mm, vias 1 -> 2

Commit message: panel
Routing:
- net GND: track 0.00 -> 0.95 mm
