File: clock-pcb/sub-boards/7-seg-display/7-seg-display.kicad_pcb (KiCad board)
At the start: 2 copper layers, 66.3 x 27.3 mm, 7 parts, among them J1 Conn_01x04_Socket, J2 Conn_01x04_Socket, U1 CC56-12EWA, U2 AS1115-BSST

Commit message: touch slider pcb
Changed lines of the file:
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@@
 	(segment
 		(start 134.2903 84.678)
-		(end 133.9776 84.3653)
-		(width 0.25)
-		(layer "F.Cu")
-		(net 3)
-	)
-	(segment
-		(start 129.1197 92.8582)
-		(end 129.1201 92.8582)
-		(width 0.25)
-		(layer "F.Cu")
-		(net 3)
-	)
-	(segment
-		(start 128.5696 92.3105)
-		(end 129.1185 92.8594)
+		(end 157.21 84.678)
 		(width 0.25)
 		(layer "F.Cu")
@@
 	(segment
 		(start 96.89 92.3105)
-		(end 128.5696 92.3105)
-		(width 0.25)
-		(layer "F.Cu")
-		(net 3)
-	)
-	(segment
-		(start 129.1185 92.8594)
-		(end 129.1197 92.8582)
-		(width 0.25)
-		(layer "F.Cu")
-		(net 3)
-	)
-	(segment
-		(start 157.21 84.678)
+		(end 129.7405 92.3105)
+		(width 0.25)
+		(layer "F.Cu")
+		(net 3)
+	)
+	(segment
+		(start 129.7405 92.3105)
+		(end 129.91 92.48)
+		(width 0.25)
+		(layer "F.Cu")
+		(net 3)
+	)
+	(segment
+		(start 132.9 84.68)
+		(end 134.2883 84.68)
+		(width 0.25)
+		(layer "F.Cu")
+		(net 3)
+	)
+	(segment
+		(start 134.2883 84.68)
 		(end 134.2903 84.678)
 		(width 0.25)
@@
 	)
 	(via
-		(at 133.9776 84.3653)
+		(at 132.9 84.68)
 		(size 0.56)
 		(drill 0.3)
@@
 	)
 	(via
-		(at 129.1201 92.8582)
+		(at 129.91 92.48)
 		(size 0.56)
 		(drill 0.3)
@@
 	)
 	(segment
-		(start 129.1201 92.8582)
-		(end 129.9075 92.0708)
+		(start 129.91 92.48)
+		(end 129.91 92.0733)
+		(width 0.25)
+		(layer "B.Cu")
+		(net 3)
+	)
+	(segment
+		(start 132.9 84.68)
+		(end 132.9 85.4429)
 		(width 0.25)
 		(layer "B.Cu")
@@
 	)
 	(segment
+		(start 132.9 85.4429)
+		(end 129.9075 88.4354)
+		(width 0.25)
+		(layer "B.Cu")
+		(net 3)
+	)
+	(segment
+		(start 129.91 92.0733)
+		(end 129.9075 92.0708)
+		(width 0.25)
+		(layer "B.Cu")
+		(net 3)
+	)
+	(segment
 		(start 129.9075 88.4354)
 		(end 129.9075 91.128)
-		(width 0.25)
-		(layer "B.Cu")
-		(net 3)
-	)
-	(segment
-		(start 133.9776 84.3653)
-		(end 129.9075 88.4354)
 		(width 0.25)
 		(layer "B.Cu")
@@
 	)
 	(segment
-		(start 123.83 79.61)
-		(end 124.1925 79.9725)
-		(width 0.25)
-		(layer "B.Cu")
-		(net 6)
-	)
-	(segment
-		(start 121.8128 79.61)
-		(end 123.83 79.61)
-		(width 0.25)
-		(layer "B.Cu")
-		(net 6)
-	)
-	(segment
-		(start 120.6948 80.728)
-		(end 121.8128 79.61)
-		(width 0.25)
-		(layer "B.Cu")
-		(net 6)
-	)
-	(segment
-		(start 124.2008 81.128131)
-		(end 124.28 81.207331)
-		(width 0.25)
-		(layer "B.Cu")
-		(net 6)
-	)
-	(segment
-		(start 124.1925 79.9725)
-		(end 124.1925 80.319569)
-		(width 0.25)
-		(layer "B.Cu")
-		(net 6)
-	)
-	(segment
-		(start 124.28 81.207331)
-		(end 124.28 85.7655)
-		(width 0.25)
-		(layer "B.Cu")
-		(net 6)
-	)
-	(segment
-		(start 124.2008 80.327869)
-		(end 124.2008 81.128131)
-		(width 0.25)
-		(layer "B.Cu")
-		(net 6)
-	)
-	(segment
 		(start 124.28 85.7655)
 		(end 124.1925 85.853)
@@
 	)
 	(segment
-		(start 124.1925 80.319569)
-		(end 124.2008 80.327869)
-		(width 0.25)
-		(layer "B.Cu")
+		(start 121.9228 79.5)
+		(end 123.72 79.5)
+		(width 0.25)
+		(layer "B.Cu")
+		(net 6)
+	)
+	(segment
+		(start 123.72 79.5)
+		(end 124.28 80.06)
+		(width 0.25)
+		(layer "B.Cu")
+		(net 6)
+	)
+	(segment
+		(start 120.6948 80.728)
+		(end 121.9228 79.5)
+		(width 0.25)
+		(layer "B.Cu")
+		(net 6)
+	)
+	(segment
+		(start 124.28 80.06)
+		(end 124.28 85.7655)
+		(width 0.25)
+		(layer "B.Cu")
