File: clock-pcb/sub-boards/side-board/side-board.kicad_pcb (KiCad board)
At the start: 2 copper layers, 51 x 18.3 mm, 4 parts, among them J1 Conn_01x07_Socket, U1 TMAG5231C1GQDBZR

Commit message: new pcb
Connections:
- net GPIO14 renamed BUTTON_EXIT
- net GPIO15 renamed BUTON_CONF
- net GPIO35 renamed HALL_SENS
Changed lines of the file:
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@@
 (kicad_pcb
-	(version 20240108)
+	(version 20241229)
 	(generator "pcbnew")
-	(generator_version "8.0")
+	(generator_version "9.0")
 	(general
 		(thickness 1.6)
@@
 	(layers
 		(0 "F.Cu" signal)
-		(31 "B.Cu" signal)
-		(32 "B.Adhes" user "B.Adhesive")
-		(33 "F.Adhes" user "F.Adhesive")
-		(34 "B.Paste" user)
-		(35 "F.Paste" user)
-		(36 "B.SilkS" user "B.Silkscreen")
-		(37 "F.SilkS" user "F.Silkscreen")
-		(38 "B.Mask" user)
-		(39 "F.Mask" user)
-		(40 "Dwgs.User" user "User.Drawings")
-		(41 "Cmts.User" user "User.Comments")
-		(42 "Eco1.User" user "User.Eco1")
-		(43 "Eco2.User" user "User.Eco2")
-		(44 "Edge.Cuts" user)
-		(45 "Margin" user)
-		(46 "B.CrtYd" user "B.Courtyard")
-		(47 "F.CrtYd" user "F.Courtyard")
-		(48 "B.Fab" user)
-		(49 "F.Fab" user)
-		(50 "User.1" user)
-		(51 "User.2" user)
-		(52 "User.3" user)
-		(53 "User.4" user)
-		(54 "User.5" user)
-		(55 "User.6" user)
-		(56 "User.7" user)
-		(57 "User.8" user)
-		(58 "User.9" user)
+		(2 "B.Cu" signal)
+		(9 "F.Adhes" user "F.Adhesive")
+		(11 "B.Adhes" user "B.Adhesive")
+		(13 "F.Paste" user)
+		(15 "B.Paste" user)
+		(5 "F.SilkS" user "F.Silkscreen")
+		(7 "B.SilkS" user "B.Silkscreen")
+		(1 "F.Mask" user)
+		(3 "B.Mask" user)
+		(17 "Dwgs.User" user "User.Drawings")
+		(19 "Cmts.User" user "User.Comments")
+		(21 "Eco1.User" user "User.Eco1")
+		(23 "Eco2.User" user "User.Eco2")
+		(25 "Edge.Cuts" user)
+		(27 "Margin" user)
+		(31 "F.CrtYd" user "F.Courtyard")
+		(29 "B.CrtYd" user "B.Courtyard")
+		(35 "F.Fab" user)
+		(33 "B.Fab" user)
+		(39 "User.1" user)
+		(41 "User.2" user)
+		(43 "User.3" user)
+		(45 "User.4" user)
+		(47 "User.5" user)
+		(49 "User.6" user)
+		(51 "User.7" user)
+		(53 "User.8" user)
+		(55 "User.9" user)
 	)
 	(setup
@@
 		(pad_to_mask_clearance 0)
 		(allow_soldermask_bridges_in_footprints no)
+		(tenting front back)
 		(pcbplotparams
-			(layerselection 0x00010fc_ffffffff)
-			(plot_on_all_layers_selection 0x0000000_00000000)
+			(layerselection 0x00000000_00000000_55555555_5755f5ff)
+			(plot_on_all_layers_selection 0x00000000_00000000_00000000_00000000)
 			(disableapertmacros no)
 			(usegerberextensions no)
@@
 			(svgprecision 4)
 			(plotframeref no)
-			(viasonmask no)
 			(mode 1)
 			(useauxorigin no)
@@
 			(pdf_front_fp_property_popups yes)
 			(pdf_back_fp_property_popups yes)
+			(pdf_metadata yes)
+			(pdf_single_document no)
 			(dxfpolygonmode yes)
 			(dxfimperialunits yes)
@@
 			(psnegative no)
 			(psa4output no)
-			(plotreference yes)
-			(plotvalue yes)
-			(plotfptext yes)
-			(plotinvisibletext no)
+			(plot_black_and_white yes)
 			(sketchpadsonfab no)
+			(plotpadnumbers no)
+			(hidednponfab no)
+			(sketchdnponfab yes)
+			(crossoutdnponfab yes)
 			(subtractmaskfromsilk no)
 			(outputformat 1)
@@
 	(net 1 "GND")
 	(net 2 "+3V3")
-	(net 3 "GPIO14")
+	(net 3 "BUTTON_EXIT")
 	(net 4 "SCL")
-	(net 5 "GPIO35")
+	(net 5 "HALL_SENS")
 	(net 6 "SDA")
-	(net 7 "GPIO15")
+	(net 7 "BUTON_CONF")
 	(footprint "clock:B3F-4055"
 		(layer "F.Cu")
@@
 			)
 		)
-		(property "Footprint" "clock:B3F-4055"
-			(at 0 0 90)
-			(layer "F.Fab")
-			(hide yes)
-			(effects
-				(font
-					(size 1.27 1.27)
-					(thickness 0.15)
-				)
-			)
-		)
 		(property "Datasheet" "https://omronfs.omron.com/en_US/ecb/products/pdf/en-b3f.pdf"
 			(at 0 0 90)
@@
 			)
 		)
-		(sheetname "Root")
+		(sheetname "/")
 		(sheetfile "side-board.kicad_sch")
 		(attr through_hole)
@@
 				(type solid)
 			)
-			(fill none)
+			(fill no)
 			(layer "F.SilkS")
 		)
@@
 			(layers "*.Cu" "*.Mask")
 			(remove_unused_layers no)
-			(net 7 "GPIO15")
+			(net 7 "BUTON_CONF")
 			(pinfunction "NO_1")
 			(pintype "passive")
@@
 			(layers "*.Cu" "*.Mask")
 			(remove_unused_layers no)
-			(net 7 "GPIO15")
+			(net 7 "BUTON_CONF")
 			(pinfunction "NO_2")
 			(pintype "passive")
 		)
+		(embedded_fonts no)
 		(model "${KIPRJMOD}/../../3D/B3F-5050.stp"
 			(offset
@@
 			)
 		)
-		(property "Footprint" "Package_TO_SOT_SMD:SOT-23-3"
-			(at 0 0 90)
-			(layer "F.Fab")
-			(hide yes)
-			(effects
-				(font
-					(size 1.27 1.27)
-					(thickness 0.15)
-				)
-			)
-		)
 		(property "Datasheet" "TMAG5231C1GQDBZR"
 			(at 0 0 90)
@@
 		)
 		(property ki_fp_filters "SOT-23-3_DBZ_TEX SOT-23-3_DBZ_TEX-M SOT-23-3_DBZ_TEX-L")
-		(sheetname "Root")
+		(sheetname "/")
 		(sheetfile "side-board.kicad_sch")
 		(attr smd)
@@
 				(type solid)
 			)
-			(fill solid)
+			(fill yes)
 			(layer "F.SilkS")
 		)
@@
 			(at -1.1375 -0.95 90)
 			(size 1.325 0.6)
-			(layers "F.Cu" "F.Paste" "F.Mask")
+			(layers "F.Cu" "F.Mask" "F.Paste")
 			(roundrect_rratio 0.25)
 			(net 2 "+3V3")
@@
 			(at -1.1375 0.95 90)
 			(size 1.325 0.6)
-			(layers "F.Cu" "F.Paste" "F.Mask")
+			(layers "F.Cu" "F.Mask" "F.Paste")
 			(roundrect_rratio 0.25)
-			(net 5 "GPIO35")
+			(net 5 "HALL_SENS")
 			(pinfunction "OUT")
 			(pintype "output")
@@
 			(at 1.1375 0 90)
 			(size 1.325 0.6)
-			(layers "F.Cu" "F.Paste" "F.Mask")
+			(layers "F.Cu" "F.Mask" "F.Paste")
 			(roundrect_rratio 0.25)
 			(net 1 "GND")
@@
 			(pintype "power_out")
 		)
+		(embedded_fonts no)
 		(model "${KICAD8_3DMODEL_DIR}/Package_TO_SOT_SMD.3dshapes/SOT-23-3.wrl"
 			(offset
@@
 			)
 		)
-		(property "Footprint" "clock:B3F-4055"
-			(at 0 0 90)
-			(layer "F.Fab")
-			(hide yes)
-			(effects
-				(font
-					(size 1.27 1.27)
-					(thickness 0.15)
-				)
-			)
-		)
 		(property "Datasheet" "https://omronfs.omron.com/en_US/ecb/products/pdf/en-b3f.pdf"
 			(at 0 0 90)
@@
 			)
 		)
-		(sheetname "Root")
+		(sheetname "/")
 		(sheetfile "side-board.kicad_sch")
 		(attr through_hole)
@@
 				(type solid)
 			)
-			(fill none)
+			(fill no)
 			(layer "F.SilkS")
 		)
@@
 			(layers "*.Cu" "*.Mask")
 			(remove_unused_layers no)
-			(net 3 "GPIO14")
+			(net 3 "BUTTON_EXIT")
 			(pinfunction "NO_1")
 			(pintype "passive")
@@
 			(layers "*.Cu" "*.Mask")
 			(remove_unused_layers no)
-			(net 3 "GPIO14")
+			(net 3 "BUTTON_EXIT")
 			(pinfunction "NO_2")
 			(pintype "passive")
 		)
+		(embedded_fonts no)
 		(model "${KIPRJMOD}/../../3D/B3F-5050.stp"
 			(offset
@@
 			)
 		)
-		(property "Footprint" "Connector_PinHeader_2.54mm:PinHeader_1x07_P2.54mm_Horizontal"
-			(at 0 0 0)
-			(unlocked yes)
-			(layer "B.Fab")
-			(hide yes)
-			(effects
-				(font
-					(size 1.27 1.27)
-					(thickness 0.15)
-				)
-				(justify mirror)
-			)
-		)
-		(property "Datasheet" ""
+		(property "Datasheet" "~"
 			(at 0 0 0)
 			(unlocked yes)
@@
 		)
 		(property ki_fp_filters "Connector*:*_1x??_*")
-		(sheetname "Root")
+		(sheetname "/")
 		(sheetfile "side-board.kicad_sch")
 		(attr through_hole)
@@
 			(layers "*.Cu" "*.Mask")
 			(remove_unused_layers no)
-			(net 5 "GPIO35")
+			(net 5 "HALL_SENS")
 			(pinfunction "Pin_3")
 			(pintype "passive")
@@
 			(layers "*.Cu" "*.Mask")
 			(remove_unused_layers no)
-			(net 3 "GPIO14")
+			(net 3 "BUTTON_EXIT")
 			(pinfunction "Pin_4")
 			(pintype "passive")
@@
 			(layers "*.Cu" "*.Mask")
 			(remove_unused_layers no)
-			(net 7 "GPIO15")
+			(net 7 "BUTON_CONF")
 			(pinfunction "Pin_5")
 			(pintype "passive")
@@
 			(pintype "passive")
 		)
+		(embedded_fonts no)
 		(model "${KICAD8_3DMODEL_DIR}/Connector_PinHeader_2.54mm.3dshapes/PinHeader_1x07_P2.54mm_Horizontal.wrl"
 			(offset
@@
 			(type default)
 		)
-		(fill none)
+		(fill no)
 		(layer "Edge.Cuts")
 	)
@@
 		(net 1)
 		(net_name "GND")
-		(layers "F&B.Cu")
+		(layers "F.Cu" "B.Cu")
 		(hatch edge 0.5)
 		(connect_pads
@@
 		(members "254b142f-a4c6-465d-8de9-bd7bd2ffa296" "ecf8d211-572a-4b17-a587-340a7ab71451")
 	)
+	(embedded_fonts no)
 )

Commit message: routing
Connections:
- S1 pad 1: GND -> +3V3
- S1 pad 2: GND -> +3V3
- S2 pad 1: GND -> +3V3
- S2 pad 2: GND -> +3V3
Routing:
- net +3V3: track 43.4 -> 71.5 mm
Changed lines of the file:
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@@
 			(layers "*.Cu" "*.Mask")
 			(remove_unused_layers no)
-			(net 1 "GND")
+			(net 2 "+3V3")
 			(pinfunction "COM_1")
 			(pintype "passive")
@@
 			(layers "*.Cu" "*.Mask")
 			(remove_unused_layers no)
-			(net 1 "GND")
+			(net 2 "+3V3")
 			(pinfunction "COM_2")
 			(pintype "passive")
@@
 			(layers "*.Cu" "*.Mask")
 			(remove_unused_layers no)
-			(net 1 "GND")
+			(net 2 "+3V3")
 			(pinfunction "COM_1")
 			(pintype "passive")
@@
 			(layers "*.Cu" "*.Mask")
 			(remove_unused_layers no)
-			(net 1 "GND")
+			(net 2 "+3V3")
 			(pinfunction "COM_2")
 			(pintype "passive")
@@
 	)
 	(segment
+		(start 113.37 55.8544)
+		(end 126.29 55.8544)
+		(width 0.2)
+		(layer "F.Cu")
+		(net 2)
+	)
+	(segment
 		(start 99.6361 55.8544)
+		(end 113.37 55.8544)
+		(width 0.2)
+		(layer "F.Cu")
+		(net 2)
+	)
+	(segment
+		(start 113.37 54.5285)
+		(end 113.555 54.3435)
+		(width 0.2)
+		(layer "F.Cu")
+		(net 2)
+	)
+	(segment
+		(start 113.37 55.8544)
+		(end 113.37 54.5285)
+		(width 0.2)
+		(layer "F.Cu")
+		(net 2)
+	)
+	(segment
+		(start 126.29 55.8544)
 		(end 132.9219 55.8544)
 		(width 0.2)
@@
 		(net 2)
 	)
+	(segment
+		(start 126.29 54.4185)
+		(end 126.355 54.3535)
+		(width 0.2)
+		(layer "F.Cu")
+		(net 2)
+	)
+	(segment
+		(start 126.29 55.8544)
+		(end 126.29 54.4185)
+		(width 0.2)
+		(layer "F.Cu")
+		(net 2)
+	)
+	(segment
+		(start 126.355 54.3535)
+		(end 126.355 66.8535)
+		(width 0.2)
+		(layer "B.Cu")
+		(net 2)
+	)
+	(segment
+		(start 113.555 54.3435)
+		(end 113.555 66.8435)
+		(width 0.2)
+		(layer "B.Cu")
+		(net 2)
+	)

Commit message: touch slider pcb
Parts:
- added R1: 10K, Resistor_SMD:R_0402_1005Metric, F.Cu at (101.2, 64.2)
- added R11: 10K, Resistor_SMD:R_0402_1005Metric, F.Cu at (100.0, 64.2)
Connections:
- S1 pad 1: +3V3 -> GND
- S1 pad 2: +3V3 -> GND
- S2 pad 1: +3V3 -> GND
- S2 pad 2: +3V3 -> GND
Routing:
- net +3V3: track 71.5 -> 58.2 mm, vias 0 -> 3
- net BUTON_CONF: track 22.7 -> 25.8 mm
- net BUTTON_EXIT: track 39.0 -> 40.1 mm
- net GND: track 0.00 -> 0.82 mm

Commit message: panel
Routing:
- net GND: vias 0 -> 128
