File: clock-pcb/sub-boards/top-board/top-board.kicad_sch (KiCad schematic)
At the start: 19 parts, among them J1 Conn_01x07_Socket, J2 Conn_01x01_Pin, U1 BH1750FVI-TR, U3 OPT3004DTSR, U4 SHT4x

Commit message: new pcb
Parts:
- removed J2: Conn_01x01_Pin, Connector_PinHeader_2.54mm:PinHeader_1x01_P2.54mm_Vertical, symbol clock:Conn_01x01_Pin
Connections:
- net GPIO25: no longer J1.5 (Pin_5)
- net GPIO26 renamed BUZZER
- net GPIO39 renamed SUB_TOP_3
- new net SUB_TOP_1: J1.5 (Pin_5)
Changed lines of the file:
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@@
 (kicad_sch
-	(version 20231120)
+	(version 20250114)
 	(generator "eeschema")
-	(generator_version "8.0")
+	(generator_version "9.0")
 	(paper "A4")
+	(text "Light Sensors"
+		(exclude_from_sim no)
+		(at 161.798 91.44 0)
+		(effects
+			(font
+				(size 1.27 1.27)
+			)
+		)
+	)
+	(text "humidity/temp sensor"
+		(exclude_from_sim no)
+		(at 90.932 42.672 0)
+		(effects
+			(font
+				(size 1.27 1.27)
+			)
+		)
+	)
+	(text "Connector"
+		(exclude_from_sim no)
+		(at 39.878 43.18 0)
+		(effects
+			(font
+				(size 1.27 1.27)
+			)
+		)
+	)
+	(text "Buzzer"
+		(exclude_from_sim no)
+		(at 148.59 42.926 0)
+		(effects
+			(font
+				(size 1.27 1.27)
+			)
+		)
+	)
 	(junction
 		(at 63.5 57.15)
@@
 		)
 	)
-	(polyline
-		(pts
-			(xy 170.18 12.7) (xy 170.18 44.45)
-		)
-		(stroke
-			(width 0)
-			(type dash)
-		)
-	)
 	(wire
 		(pts
@@
 		)
 	)
-	(text "Light Sensors"
-		(exclude_from_sim no)
-		(at 161.798 91.44 0)
-		(effects
-			(font
-				(size 1.27 1.27)
-			)
-		)
-	)
-	(text "humidity/temp sensor"
-		(exclude_from_sim no)
-		(at 90.932 42.672 0)
-		(effects
-			(font
-				(size 1.27 1.27)
-			)
-		)
-	)
-	(text "Connector"
-		(exclude_from_sim no)
-		(at 39.878 43.18 0)
-		(effects
-			(font
-				(size 1.27 1.27)
-			)
-		)
-	)
-	(text "Buzzer"
-		(exclude_from_sim no)
-		(at 148.59 42.926 0)
-		(effects
-			(font
-				(size 1.27 1.27)
-			)
-		)
-	)
-	(global_label "GPIO26"
+	(global_label "SCL"
 		(shape input)
-		(at 115.57 29.21 180)
+		(at 30.48 67.31 180)
 		(fields_autoplaced yes)
 		(effects
@@
 		)
 		(property "Intersheetrefs" "${INTERSHEET_REFS}"
-			(at 105.6905 29.21 0)
+			(at 23.9872 67.31 0)
 			(effects
 				(font
@@
 		)
 	)
-	(global_label "SCL"
+	(global_label "SUB_TOP_3"
 		(shape input)
-		(at 30.48 67.31 180)
+		(at 31.75 29.21 90)
 		(fields_autoplaced yes)
 		(effects
@@
 				(size 1.27 1.27)
 			)
-			(justify right)
+			(justify left)
 		)
 		(property "Intersheetrefs" "${INTERSHEET_REFS}"
-			(at 23.9872 67.31 0)
+			(at 31.75 15.702 90)
 			(effects
 				(font
 					(size 1.27 1.27)
 				)
-				(justify right)
+				(justify left)
 				(hide yes)
 			)
 		)
 	)
-	(global_label "GPIO39"
+	(global_label "SDA"
 		(shape input)
-		(at 31.75 29.21 90)
+		(at 85.09 57.15 90)
 		(fields_autoplaced yes)
 		(effects
@@
 		)
 		(property "Intersheetrefs" "${INTERSHEET_REFS}"
-			(at 31.75 19.3305 90)
+			(at 85.09 50.5967 90)
 			(effects
 				(font
@@
 		)
 	)
-	(global_label "SDA"
+	(global_label "SCL"
 		(shape input)
-		(at 85.09 57.15 90)
+		(at 90.17 57.15 90)
 		(fields_autoplaced yes)
 		(effects
@@
 		)
 		(property "Intersheetrefs" "${INTERSHEET_REFS}"
-			(at 85.09 50.5967 90)
+			(at 90.17 50.6572 90)
 			(effects
 				(font
@@
 		)
 	)
-	(global_label "SCL"
+	(global_label "BUZZER"
 		(shape input)
-		(at 90.17 57.15 90)
+		(at 115.57 29.21 180)
 		(fields_autoplaced yes)
 		(effects
@@
 				(size 1.27 1.27)
 			)
-			(justify left)
+			(justify right)
 		)
 		(property "Intersheetrefs" "${INTERSHEET_REFS}"
-			(at 90.17 50.6572 90)
+			(at 105.1463 29.21 0)
 			(effects
 				(font
 					(size 1.27 1.27)
 				)
-				(justify left)
+				(justify right)
 				(hide yes)
 			)
@@
 		)
 	)
-	(global_label "GPIO25"
+	(global_label "SUB_TOP_1"
 		(shape input)
 		(at 26.67 29.21 90)
@@
 		)
 		(property "Intersheetrefs" "${INTERSHEET_REFS}"
-			(at 26.67 19.3305 90)
+			(at 26.67 15.702 90)
 			(effects
 				(font
@@
 		)
 	)
-	(global_label "GPIO39"
-		(shape input)
-		(at 162.56 27.94 90)
-		(fields_autoplaced yes)
-		(effects
-			(font
-				(size 1.27 1.27)
-			)
-			(justify left)
-		)
-		(property "Intersheetrefs" "${INTERSHEET_REFS}"
-			(at 162.56 18.0605 90)
-			(effects
-				(font
-					(size 1.27 1.27)
-				)
-				(justify left)
-				(hide yes)
-			)
-		)
-	)
-	(global_label "GPIO26"
+	(global_label "BUZZER"
 		(shape input)
 		(at 29.21 29.21 90)
@@
 		)
 		(property "Intersheetrefs" "${INTERSHEET_REFS}"
-			(at 29.21 19.3305 90)
+			(at 29.21 18.7863 90)
 			(effects
 				(font
@@
 	)
 	(symbol
-		(lib_id "clock:Conn_01x01_Pin")
-		(at 162.56 33.02 90)
-		(unit 1)
-		(exclude_from_sim no)
-		(in_bom yes)
-		(on_board yes)
-		(dnp no)
-		(fields_autoplaced yes)
-		(property "Reference" "J2"
-			(at 163.83 31.1149 90)
-			(effects
-				(font
-					(size 1.27 1.27)
-				)
-				(justify right)
-			)
-		)
-		(property "Value" "Conn_01x01_Pin"
-			(at 163.83 33.6549 90)
-			(effects
-				(font
-					(size 1.27 1.27)
-				)
-				(justify right)
-				(hide yes)
-			)
-		)
-		(property "Footprint" "Connector_PinHeader_2.54mm:PinHeader_1x01_P2.54mm_Vertical"
-			(at 162.56 33.02 0)
-			(effects
-				(font
-					(size 1.27 1.27)
-				)
-				(hide yes)
-			)
-		)
-		(property "Datasheet" "~"
-			(at 162.56 33.02 0)
-			(effects
-				(font
-					(size 1.27 1.27)
-				)
-				(hide yes)
-			)
-		)
-		(property "Description" "Generic connector, single row, 01x01, script generated"
-			(at 162.56 33.02 0)
-			(effects
-				(font
-					(size 1.27 1.27)
-				)
-				(hide yes)
-			)
-		)
-		(pin "1"
-		)
-		(instances
-			(project ""
-				(path "/b1deab82-097c-4ad9-80a9-eb8517127baf"
-					(reference "J2")
-					(unit 1)
-				)
-			)
-		)
-	)
-	(symbol
 		(lib_id "clock:LTR-F216A")
 		(at 87.63 66.04 0)
@@
 		)
 	)
+	(embedded_fonts no)
 )

Commit message: routing
Parts:
- removed C2, C5: 0.1uF, Capacitor_SMD:C_0603_1608Metric, symbol clock:C
- removed JP2: SolderJumper_3_Bridged12, Jumper:SolderJumper-3_P1.3mm_Bridged2Bar12_RoundedPad1.0x1.5mm, symbol clock:SolderJumper_3_Bridged12
- removed R3: 10K, Resistor_SMD:R_0402_1005Metric, symbol clock:R
- removed U1: BH1750FVI-TR, clock:XDCR_BH1750FVI-TR, symbol clock:BH1750FVI-TR
- removed U3: OPT3004DTSR, clock:DNP6_TEX, symbol clock:OPT3004DTSR
- added IC1: VEML6030-GS15, clock:VEML6030GS15, symbol VEML6030-GS15:VEML6030-GS15
- added LS1: Speaker_Crystal, clock:AST0760_MAL, symbol Device:Speaker_Crystal
- R1: value 1K -> 10K
Connections:
- net +3V3: now also C1.2, R1.1, IC1.6 (VDD); no longer R1.2
- net GND: now also C1.1, IC1.1 (GND), LS1.2; no longer C1.2
- net GPIO25: now also R1.2, IC1.3 (INT)
- net SCL: now also IC1.5 (SCL)
- net SDA: now also IC1.2 (SDA)
- net at JP1.2 (C): now also IC1.4 (ADDR)
- net BUZZER_IN: now reaches L1.1, R4.1
- net BUZZER_IN: now also LS1.1
Other:
- note added: "Buzzers"
- note removed: "Buzzer"
- moved on the sheet: L1, R4

Commit message: touch slider pcb
Parts:
- added C2: 0.1uF, Capacitor_SMD:C_0603_1608Metric, symbol clock:C
- added JP2: SolderJumper_3_Bridged12, Jumper:SolderJumper-3_P1.3mm_Bridged2Bar12_RoundedPad1.0x1.5mm, symbol clock:SolderJumper_3_Bridged12
- added U1: BMP280, Package_LGA:Bosch_LGA-8_2x2.5mm_P0.65mm_ClockwisePinNumbering, symbol Sensor_Pressure:BMP280
Connections:
- net +3V3: now also C2.2, JP2.3 (B), U1.2 (CSB), U1.6 (VDDIO), U1.8 (VDD)
- net GND: now also C2.1, JP2.1 (A), U1.1 (GND), U1.7 (GND)
- net SCL: now also U1.4 (SCK)
- net SDA: now also U1.3 (SDI)
- new net: JP2.2 (C), U1.5 (SDO)

Commit message: panel
Parts:
- added C13, C5: 1uF, Capacitor_SMD:C_0603_1608Metric, symbol Watchy:C
- added C7: 100uF, Capacitor_THT:CP_Radial_D5.0mm_P2.50mm, symbol Device:C_Polarized
- added R3: 10K, Resistor_SMD:R_0402_1005Metric, symbol clock:R
- added R5: 22R, Resistor_SMD:R_0402_1005Metric, symbol clock:R
- added R6: 22R, Resistor_THT:R_Axial_DIN0204_L3.6mm_D1.6mm_P2.54mm_Vertical, symbol clock:R
- added U3: APDS-9960, clock:Avago_APDS-9960, symbol Sensor:APDS-9960
- U1: footprint Package_LGA:Bosch_LGA-8_2x2.5mm_P0.65mm_ClockwisePinNumbering -> clock:Bosch_LGA-8_2x2.5mm_P0.65mm_ClockwisePinNumbering
Connections:
- net GPIO25 is gone; now on net SUB_TOP_1: IC1.3 (INT), R1.2, R2.2, U2.5 (INT)
- net +3V3: now also C13.1, C7.1, R3.1, R5.1, R6.1, U3.5 (LED_A)
- net GND: now also C13.2, C5.2, C7.2, U3.6 (GND)
- net SCL: now also U3.7 (SCL)
- net SDA: now also U3.1 (SDA)
- net SUB_TOP_3: now also R3.2, U3.2 (INT)
- new net: C5.1, R5.2, R6.2, U3.8 (VDD)
- new net: U3.3 (LDR), U3.4 (LED_K)
