File: clock-pcb/sub-boards/top-board/top-board.kicad_pcb (KiCad board)
At the start: 2 copper layers, 51 x 18.3 mm, 19 parts, among them J1 Conn_01x07_Socket, J2 Conn_01x01_Pin, U1 BH1750FVI-TR, U3 OPT3004DTSR, U4 SHT4x

Commit message: new pcb
Parts:
- removed J2: Conn_01x01_Pin, Connector_PinHeader_2.54mm:PinHeader_1x01_P2.54mm_Vertical
Connections:
- net GPIO26 renamed BUZZER
- J1 pad 3: GPIO39 -> SUB_TOP_3
- J1 pad 5: GPIO25 -> SUB_TOP_1
Routing:
- net GPIO39: track 10.8 -> 0.00 mm

Commit message: routing
Parts:
- removed C2, C5: 0.1uF, Capacitor_SMD:C_0603_1608Metric
- removed JP2: SolderJumper_3_Bridged12, Jumper:SolderJumper-3_P1.3mm_Bridged2Bar12_RoundedPad1.0x1.5mm
- removed R3: 10K, Resistor_SMD:R_0402_1005Metric
- removed U1: BH1750FVI-TR, clock:XDCR_BH1750FVI-TR
- removed U3: OPT3004DTSR, clock:DNP6_TEX
- added IC1: VEML6030-GS15, clock:VEML6030GS15, F.Cu at (109.7, 60.2)
- added LS1: Speaker_Crystal, clock:AST0760_MAL, F.Cu at (121.9, 60.2)
- R1: value 1K -> 10K
- R4: moved to F.Cu
- moved R4 14.3 mm to (108.4, 54.7)
- moved C1 10.7 mm to (112.4, 60.2), turned to -90 degrees
- moved JP1 8.79 mm to (109.7, 63.7)
- moved R1 8.02 mm to (109.0, 57.1), turned to -90 degrees
- moved R2 2.91 mm to (103.9, 57.1)
- moved C3 2.90 mm to (103.9, 62.8)
- moved C4 2.90 mm to (103.9, 64.3)
- moved U2 2.90 mm to (103.9, 60.2)
- moved U4 0.94 mm to (139.0, 60.1)
- moved C6 0.94 mm to (141.0, 60.1)
Connections:
- net Net-(L1-Pad1) renamed BUZZER_IN
- C1 pad 1: Net-(U1-DVI) -> GND
- C1 pad 2: GND -> +3V3
- R1 pad 1: Net-(U1-DVI) -> +3V3
- R1 pad 2: +3V3 -> GPIO25
Routing:
- net BUZZER_IN: track 2.14 -> 19.7 mm, vias 0 -> 2
- net BUZZER: track 25.6 -> 12.5 mm, vias 0 -> 1
- net GPIO25: track 19.4 -> 8.36 mm, vias 1 -> 0
- net Net-(JP2-C): track 11.0 -> 0.00 mm, vias 2 -> 0
- net SDA: track 54.5 -> 64.6 mm, vias 1 -> 2
- net +3V3: track 75.0 -> 70.1 mm
- net GND: track 4.53 -> 8.73 mm
- net SCL: track 60.2 -> 64.2 mm
- net Net-(U1-DVI): track 2.54 -> 0.00 mm
- net Net-(IC1-ADDR): track 3.67 -> 2.89 mm

Commit message: touch slider pcb
Parts:
- added C2: 0.1uF, Capacitor_SMD:C_0603_1608Metric, F.Cu at (140.8, 58.6)
- added JP2: SolderJumper_3_Bridged12, Jumper:SolderJumper-3_P1.3mm_Bridged2Bar12_RoundedPad1.0x1.5mm, F.Cu at (140.7, 53.2)
- added U1: BMP280, Package_LGA:Bosch_LGA-8_2x2.5mm_P0.65mm_ClockwisePinNumbering, F.Cu at (140.8, 56.2)
- moved U4 4.38 mm to (140.8, 64.1), turned to 90 degrees
- moved C6 1.52 mm to (140.8, 61.6), turned to 180 degrees
Routing:
- net SDA: track 64.6 -> 79.1 mm
- net +3V3: track 70.1 -> 84.3 mm
- net Net-(JP2-C): track 0.00 -> 9.92 mm, vias 0 -> 2
- net SCL: track 64.2 -> 73.7 mm, vias 3 -> 1
- net GND: track 8.73 -> 10.7 mm, vias 3 -> 12
- net Net-(IC1-ADDR): track 2.89 -> 3.44 mm

Commit message: panel
Parts:
- added C13: 1uF, Capacitor_SMD:C_0603_1608Metric, F.Cu at (99.9, 60.2)
- added C5: 1uF, Capacitor_SMD:C_0603_1608Metric, F.Cu at (106.3, 60.3)
- added C7: 100uF, Capacitor_THT:CP_Radial_D5.0mm_P2.50mm, B.Cu at (101.4, 63.2)
- added R3: 10K, Resistor_SMD:R_0402_1005Metric, F.Cu at (103.4, 63.5)
- added R5: 22R, Resistor_SMD:R_0402_1005Metric, F.Cu at (104.4, 57.6)
- added R6: 22R, Resistor_THT:R_Axial_DIN0204_L3.6mm_D1.6mm_P2.54mm_Vertical, B.Cu at (102.7, 55.0)
- added U3: APDS-9960, clock:Avago_APDS-9960, F.Cu at (103.0, 60.2)
- U1: footprint Package_LGA:Bosch_LGA-8_2x2.5mm_P0.65mm_ClockwisePinNumbering -> clock:Bosch_LGA-8_2x2.5mm_P0.65mm_ClockwisePinNumbering
- moved C4 9.71 mm to (113.6, 63.7), turned to 90 degrees
- moved C3 8.27 mm to (112.1, 63.7), turned to 90 degrees
- moved JP1 7.28 mm to (113.1, 57.3), turned to -90 degrees
- moved R2 7.08 mm to (106.5, 63.7), turned to 0 degrees
- moved U2 6.70 mm to (109.6, 63.7), turned to 90 degrees
- moved C1 6.48 mm to (109.6, 54.4), turned to 0 degrees
- moved IC1 2.94 mm to (109.6, 57.3), turned to 0 degrees
- moved R1 2.64 mm to (106.5, 57.9), turned to 0 degrees
- moved R4 2.62 mm to (109.5, 52.3)
- moved JP2 0.30 mm to (140.7, 52.9)
- turned C6 to 0 degrees
Connections:
- IC1 pad 3: GPIO25 -> SUB_TOP_1
- R1 pad 2: GPIO25 -> SUB_TOP_1
- R2 pad 2: GPIO25 -> SUB_TOP_1
- U2 pad 5: GPIO25 -> SUB_TOP_1
Routing:
- net SUB_TOP_1: track 0.00 -> 19.0 mm, vias 0 -> 2
- net GND: track 10.7 -> 27.4 mm, vias 12 -> 168
- net +3V3: track 84.3 -> 98.8 mm
- net SUB_TOP_3: track 0.00 -> 12.7 mm, vias 0 -> 2
- net GPIO25: track 8.37 -> 0.00 mm
- net Net-(U3-VDD): track 0.00 -> 7.86 mm, vias 0 -> 1
- net BUZZER: track 12.5 -> 16.7 mm
- net SDA: track 79.1 -> 82.9 mm, vias 2 -> 5
- net BUZZER_IN: track 19.7 -> 22.6 mm
- net SCL: track 73.7 -> 72.5 mm, vias 1 -> 0
- net Net-(U3-LDR): track 0.00 -> 0.97 mm
- net Net-(IC1-ADDR): track 3.44 -> 2.89 mm
