File: clock-pcb/sub-boards/touch-pad/touch-pad.kicad_pcb (KiCad board)
At the start: 2 copper layers, 99 x 60 mm, 6 parts, among them J1 Conn_01x01_Pin, J2 Conn_01x01_Pin, J3 Conn_01x01_Pin, J4 Conn_01x01_Pin, J5 Conn_01x01_Pin, J6 Conn_01x01_Pin

Commit message: touch slider pcb
Parts:
- added J8: Conn_01x04_Pin, clock:TouchSlider-4_90x55mm, F.Cu at (176.3, 99.3)
- J6: footprint Connector_PinHeader_2.54mm:PinHeader_1x02_P2.54mm_Vertical_SMD_Pin1Left -> Connector_PinHeader_2.54mm:PinHeader_1x01_P2.54mm_Vertical
- moved J4 75.6 mm to (160.8, 70.5)
- moved J3 74.6 mm to (207.0, 68.3)
- moved J5 67.7 mm to (176.4, 68.3)
- moved J1 61.8 mm to (146.2, 68.3)
- moved J2 52.4 mm to (190.7, 70.5)
- moved J6 52.3 mm to (131.6, 70.5)
Connections:
- net GPIO2 renamed GUARD
- J1 pad 1: GPIO4_T -> GND
- J2 pad 1: GPIO33 -> SLID_1
- J3 pad 1: GPIO32 -> GND
- J4 pad 1: GPIO27 -> SLID_0
- J6 pad 1: GND -> SLID_2
Routing:
- net SLID_2: track 0.00 -> 175.2 mm
- net SLID_1: track 0.00 -> 29.0 mm
- net SLID_0: track 0.00 -> 28.8 mm
- added copper zone on F.Cu, net GND
- added copper zone on F.Cu, net GUARD
- removed copper zone on B.Cu, net GND
Other:
- board size 99 x 60 mm -> 100 x 65 mm

Commit message: panel
Parts:
- Slid 0: renamed from J4
- Slid 1: renamed from J2
- slid 2: renamed from J6
- renumbered J1 to GND, J3 to GND, J5 to GUARD
Changed lines of the file:
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@@
 		(descr "Through hole straight pin header, 1x01, 2.54mm pitch, single row")
 		(tags "Through hole pin header THT 1x01 2.54mm single row")
-		(property "Reference" "J1"
-			(at 0 2.33 90)
+		(property "Reference" "GND"
+			(at -2.185 0.036 180)
 			(layer "B.SilkS")
 			(effects
@@
 		(descr "Through hole straight pin header, 1x01, 2.54mm pitch, single row")
 		(tags "Through hole pin header THT 1x01 2.54mm single row")
-		(property "Reference" "J2"
+		(property "Reference" "Slid 1"
 			(at 0 2.33 0)
 			(layer "B.SilkS")
@@
 		(descr "Through hole straight pin header, 1x01, 2.54mm pitch, single row")
 		(tags "Through hole pin header THT 1x01 2.54mm single row")
-		(property "Reference" "J3"
-			(at 0 2.33 0)
+		(property "Reference" "GND"
+			(at -0.0475 -2.115 0)
 			(layer "B.SilkS")
 			(effects
@@
 		(descr "Through hole straight pin header, 1x01, 2.54mm pitch, single row")
 		(tags "Through hole pin header THT 1x01 2.54mm single row")
-		(property "Reference" "J6"
-			(at 0 2.33 0)
+		(property "Reference" "slid 2"
+			(at -0.065 2.005 0)
 			(layer "B.SilkS")
 			(effects
@@
 		(descr "Through hole straight pin header, 1x01, 2.54mm pitch, single row")
 		(tags "Through hole pin header THT 1x01 2.54mm single row")
-		(property "Reference" "J4"
+		(property "Reference" "Slid 0"
 			(at 0 2.33 0)
 			(layer "B.SilkS")
@@
 		(descr "Through hole straight pin header, 1x01, 2.54mm pitch, single row")
 		(tags "Through hole pin header THT 1x01 2.54mm single row")
-		(property "Reference" "J5"
-			(at 0.87 2.33 0)
-			(layer "B.SilkS")
-			(effects
+		(property "Reference" "GUARD"
+			(at -0.06 -2.16 0)
+			(layer "B.SilkS")
+			(effects

Commit message: new pcb drafts
Parts:
- removed GND (x2), GUARD: Conn_01x01_Pin, Connector_PinHeader_2.54mm:PinHeader_1x01_P2.54mm_Vertical
- removed Slid 0: Conn_01x01_Pin, Connector_PinHeader_2.54mm:PinHeader_1x01_P2.54mm_Vertical
- removed Slid 1: Conn_01x01_Pin, Connector_PinHeader_2.54mm:PinHeader_1x01_P2.54mm_Vertical
- removed slid 2: Conn_01x01_Pin, Connector_PinHeader_2.54mm:PinHeader_1x01_P2.54mm_Vertical
- added C1: 0.1uF, Capacitor_SMD:C_0603_1608Metric, F.Cu at (183.1, 68.5)
- added C14: 1uF, Capacitor_SMD:C_0603_1608Metric, F.Cu at (181.2, 68.5)
- added C15: 1uF, Capacitor_SMD:C_0603_1608Metric, F.Cu at (184.7, 68.5)
- added J7: Conn_01x05_Pin, Connector_PinHeader_2.54mm:PinHeader_1x05_P2.54mm_Vertical, F.Cu at (202.6, 70.0)
- added JP2: SolderJumper_3_Bridged12, clock:jumper_solder_small_3_bridged, F.Cu at (170.8, 68.2)
- added R1: 100k, Resistor_SMD:R_0402_1005Metric, F.Cu at (196.0, 68.1)
- added R10: 10K, Resistor_SMD:R_0402_1005Metric, F.Cu at (172.3, 72.4)
- added R11: 10K, Resistor_SMD:R_0402_1005Metric, F.Cu at (183.1, 70.7)
- added R12: 100k, Resistor_SMD:R_0402_1005Metric, F.Cu at (197.3, 68.2)
- added R16: 10K, Resistor_SMD:R_0402_1005Metric, F.Cu at (178.8, 72.4)
- added R7: 47K, Resistor_SMD:R_0402_1005Metric, F.Cu at (179.8, 68.4)
- added R8: 10K, Resistor_SMD:R_0402_1005Metric, F.Cu at (172.3, 69.7)
- added R9: 10K, Resistor_SMD:R_0402_1005Metric, F.Cu at (167.7, 68.0)
- added U8: AT42QT2120-MMHR, clock:QFN45P300X300X85-21N, F.Cu at (176.6, 68.9)
- moved J8 2.51 mm to (176.4, 101.8), turned to 180 degrees
Routing:
- net SLID_0: track 28.8 -> 71.3 mm
- net SLID_2: track 175.2 -> 216.9 mm
- net TOUCH_INT: track 0.00 -> 37.6 mm, vias 0 -> 2
- net +3V3: track 0.00 -> 37.2 mm
- net SDA: track 0.00 -> 36.9 mm, vias 0 -> 3
- net SCL: track 0.00 -> 31.3 mm, vias 0 -> 2
- net GND: track 0.00 -> 21.8 mm, vias 0 -> 13
- net Net-(U8-~{RESET}): track 0.00 -> 16.2 mm, vias 0 -> 3
- net SLID_1: track 29.0 -> 40.0 mm
- net GUARD_RES: track 0.00 -> 8.26 mm
- net SLID_1_RES: track 0.00 -> 3.67 mm
- net SLID_0_RES: track 0.00 -> 3.64 mm
- net SLID_2_RES: track 0.00 -> 2.24 mm
- removed copper zone on F.Cu, net GUARD
